Commit message: Add Yard Force SA650ECO simulator profile

File: ros2/src/mowgli_simulation/urdf_webots/mowgli_webots.urdf (robot description, URDF)
Before this commit: robot MowgliMower, 7 links, 6 joints
Links:
- link base_link: geometry collision box size=0.57 0.39 0.26; visual box size=0.57 0.39 0.26
- link left_wheel: geometry collision cylinder length=0.04 radius=0.100; visual cylinder length=0.04 radius=0.100
- link right_wheel: geometry collision cylinder length=0.04 radius=0.100; visual cylinder length=0.04 radius=0.100
Joints:
- joint base_footprint_to_base_link: origin xyz=0 0 0.093 rpy=0 0 0 -> xyz=0 0 0.100 rpy=0 0 0
- joint base_link_to_gps: origin xyz=0.30 0 0.19 rpy=0 0 0 -> xyz=0.285 0 0.260 rpy=0 0 0
- joint base_link_to_imu: origin xyz=0.18 0 0.095 rpy=0 0 0 -> xyz=0.17 0 0.260 rpy=0 0 0
- joint base_link_to_lidar: origin xyz=0 0.024 0.390 rpy=0 0 3.1408 -> xyz=0 0.024 0.460 rpy=0 0 3.1408
- joint left_wheel_motor: origin xyz=0 0.1625 0 rpy=0 0 0 -> xyz=0 0.170 0 rpy=0 0 0
- joint right_wheel_motor: origin xyz=0 -0.1625 0 rpy=0 0 0 -> xyz=0 -0.170 0 rpy=0 0 0
